File: circuit/stm32f103_button.kicad_sch (KiCad schematic)
At the start: 12 parts, among them SW2 TL1105AF160Q, SW3 TL1105AF160Q, SW4 TL1105AF160Q, SW5 TL1105AF160Q

Commit message: V.1.0.4.0_260930
□ PinkBug Lab Study
 - STM32 : 14_E
Parts:
- renumbered R7 to R17, R8 to R18, R9 to R19, R10 to R20, R11 to R21, R12 to R22, R13 to R23, R14 to R24
Changed lines of the file:
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@@
 		(in_pos_files yes)
 		(dnp no)
-		(property "Reference" "#PWR023"
+		(property "Reference" "#PWR035"
 			(at 203.2 52.07 0)
 			(hide yes)
@@
 			(project "stm32f103_t"
 				(path "/85c6611a-7c24-4cf6-98b3-fc639d9f6ec5/72ead482-8f30-41c5-ae60-001db1b7efa5"
-					(reference "#PWR023")
+					(reference "#PWR035")
 					(unit 1)
 				)
@@
 		(in_pos_files yes)
 		(dnp no)
-		(property "Reference" "R13"
+		(property "Reference" "R23"
 			(at 200.66 55.118 90)
 			(show_name no)
@@
 			(project "stm32f103_t"
 				(path "/85c6611a-7c24-4cf6-98b3-fc639d9f6ec5/72ead482-8f30-41c5-ae60-001db1b7efa5"
-					(reference "R13")
+					(reference "R23")
 					(unit 1)
 				)
@@
 		(in_pos_files yes)
 		(dnp no)
-		(property "Reference" "#PWR021"
+		(property "Reference" "#PWR033"
 			(at 152.4 52.07 0)
 			(hide yes)
@@
 			(project "stm32f103_t"
 				(path "/85c6611a-7c24-4cf6-98b3-fc639d9f6ec5/72ead482-8f30-41c5-ae60-001db1b7efa5"
-					(reference "#PWR021")
+					(reference "#PWR033")
 					(unit 1)
 				)
@@
 		(in_pos_files yes)
 		(dnp no)
-		(property "Reference" "#PWR024"
+		(property "Reference" "#PWR036"
 			(at 203.2 85.09 0)
 			(hide yes)
@@
 			(project "stm32f103_t"
 				(path "/85c6611a-7c24-4cf6-98b3-fc639d9f6ec5/72ead482-8f30-41c5-ae60-001db1b7efa5"
-					(reference "#PWR024")
+					(reference "#PWR036")
 					(unit 1)
 				)
@@
 		(in_pos_files yes)
 		(dnp no)
-		(property "Reference" "R12"
+		(property "Reference" "R22"
 			(at 160.02 59.182 0)
 			(show_name no)
@@
 			(project "stm32f103_t"
 				(path "/85c6611a-7c24-4cf6-98b3-fc639d9f6ec5/72ead482-8f30-41c5-ae60-001db1b7efa5"
-					(reference "R12")
+					(reference "R22")
 					(unit 1)
 				)
@@
 		(in_pos_files yes)
 		(dnp no)
-		(property "Reference" "R9"
+		(property "Reference" "R19"
 			(at 99.06 55.118 90)
 			(show_name no)
@@
 			(project "stm32f103_t"
 				(path "/85c6611a-7c24-4cf6-98b3-fc639d9f6ec5/72ead482-8f30-41c5-ae60-001db1b7efa5"
-					(reference "R9")
+					(reference "R19")
 					(unit 1)
 				)
@@
 		(in_pos_files yes)
 		(dnp no)
-		(property "Reference" "R10"
+		(property "Reference" "R20"
 			(at 109.22 59.182 0)
 			(show_name no)
@@
 			(project "stm32f103_t"
 				(path "/85c6611a-7c24-4cf6-98b3-fc639d9f6ec5/72ead482-8f30-41c5-ae60-001db1b7efa5"
-					(reference "R10")
+					(reference "R20")
 					(unit 1)
 				)
@@
 		(in_pos_files yes)
 		(dnp no)
-		(property "Reference" "#PWR018"
+		(property "Reference" "#PWR030"
 			(at 50.8 85.09 0)
 			(hide yes)
@@
 			(project "stm32f103_t"
 				(path "/85c6611a-7c24-4cf6-98b3-fc639d9f6ec5/72ead482-8f30-41c5-ae60-001db1b7efa5"
-					(reference "#PWR018")
+					(reference "#PWR030")
 					(unit 1)
 				)
@@
 		(in_pos_files yes)
 		(dnp no)
-		(property "Reference" "R7"
+		(property "Reference" "R17"
 			(at 48.26 55.118 90)
 			(show_name no)
@@
 			(project "stm32f103_t"
 				(path "/85c6611a-7c24-4cf6-98b3-fc639d9f6ec5/72ead482-8f30-41c5-ae60-001db1b7efa5"
-					(reference "R7")
+					(reference "R17")
 					(unit 1)
 				)
@@
 		(in_pos_files yes)
 		(dnp no)
-		(property "Reference" "#PWR019"
+		(property "Reference" "#PWR031"
 			(at 101.6 52.07 0)
 			(hide yes)
@@
 			(project "stm32f103_t"
 				(path "/85c6611a-7c24-4cf6-98b3-fc639d9f6ec5/72ead482-8f30-41c5-ae60-001db1b7efa5"
-					(reference "#PWR019")
+					(reference "#PWR031")
 					(unit 1)
 				)
@@
 		(in_pos_files yes)
 		(dnp no)
-		(property "Reference" "R11"
+		(property "Reference" "R21"
 			(at 149.86 55.118 90)
 			(show_name no)
@@
 			(project "stm32f103_t"
 				(path "/85c6611a-7c24-4cf6-98b3-fc639d9f6ec5/72ead482-8f30-41c5-ae60-001db1b7efa5"
-					(reference "R11")
+					(reference "R21")
 					(unit 1)
 				)
@@
 		(in_pos_files yes)
 		(dnp no)
-		(property "Reference" "#PWR017"
+		(property "Reference" "#PWR029"
 			(at 50.8 52.07 0)
 			(hide yes)
@@
 			(project "stm32f103_t"
 				(path "/85c6611a-7c24-4cf6-98b3-fc639d9f6ec5/72ead482-8f30-41c5-ae60-001db1b7efa5"
-					(reference "#PWR017")
+					(reference "#PWR029")
 					(unit 1)
 				)
@@
 		(in_pos_files yes)
 		(dnp no)
-		(property "Reference" "R14"
+		(property "Reference" "R24"
 			(at 210.82 59.182 0)
 			(show_name no)
@@
 			(project "stm32f103_t"
 				(path "/85c6611a-7c24-4cf6-98b3-fc639d9f6ec5/72ead482-8f30-41c5-ae60-001db1b7efa5"
-					(reference "R14")
+					(reference "R24")
 					(unit 1)
 				)
@@
 		(in_pos_files yes)
 		(dnp no)
-		(property "Reference" "#PWR020"
+		(property "Reference" "#PWR032"
 			(at 101.6 85.09 0)
 			(hide yes)
@@
 			(project "stm32f103_t"
 				(path "/85c6611a-7c24-4cf6-98b3-fc639d9f6ec5/72ead482-8f30-41c5-ae60-001db1b7efa5"
-					(reference "#PWR020")
+					(reference "#PWR032")
 					(unit 1)
 				)
@@
 		(in_pos_files yes)
 		(dnp no)
-		(property "Reference" "R8"
+		(property "Reference" "R18"
 			(at 58.42 59.182 0)
 			(show_name no)
@@
 			(project "stm32f103_t"
 				(path "/85c6611a-7c24-4cf6-98b3-fc639d9f6ec5/72ead482-8f30-41c5-ae60-001db1b7efa5"
-					(reference "R8")
+					(reference "R18")
 					(unit 1)
 				)
@@
 		(in_pos_files yes)
 		(dnp no)
-		(property "Reference" "#PWR022"
+		(property "Reference" "#PWR034"
 			(at 152.4 85.09 0)
 			(hide yes)
@@
 			(project "stm32f103_t"
 				(path "/85c6611a-7c24-4cf6-98b3-fc639d9f6ec5/72ead482-8f30-41c5-ae60-001db1b7efa5"
-					(reference "#PWR022")
-					(unit 1)
-				)
+					(reference "#PWR034")
+					(unit 1)
+				)
