File: circuit/stm32f103_ftdi.kicad_sch (KiCad schematic)
At the start: 12 parts

Commit message: V.1.0.3.0_260928
□ PinkBug Lab Study
 - STM32 : 13
Parts:
- removed C12, C13, C14, C15: 20pF(2012), 0101_capacitor:c_0805_2012_smd, symbol 0101_capacitor:C
- removed R15, R16, R17, R18: 1kΩ(2012), 0103_resistor:r_0805_2012_smd, symbol 0103_resistor:R
- removed RV1, RV2, RV3, RV4: RK09K113004U, 0103_resistor:rk09k113004u, symbol 0103_resistor:RK09K113004U
- added C16, C18, C19: 0.1uF(2012), 0101_capacitor:c_0805_2012_smd, symbol 0101_capacitor:C
- added C17: 4.7uF(2012), 0101_capacitor:c_0805_2012_smd, symbol 0101_capacitor:C
- added D5, D6: LED(GRN), symbol 0301_led:LED
- added R21: 10kΩ(2012), 0103_resistor:r_0805_2012_smd, symbol 0103_resistor:R
- added R22, R23: 62Ω(2012), 0103_resistor:r_0805_2012_smd, symbol 0103_resistor:R
- added U3: FT232RNL, 0402_interface_communication:ft232rnl, symbol 0402_interface_communication:FT232RNL
Connections:
- net +3.3V: now also C16.2, R22.2, R23.2, U3.4 (VCCIO)
- net GND: now also C16.1, C17.1, C18.1, C19.2, U3.18 (GND), U3.21 (GND), U3.25 (AGND), U3.26 (TEST), U3.7 (GND)
- new net: C19.1, U3.17 (3V3OUT)
- new net: R21.2, U3.19 (~{RESET})
- new net: D6.2 (A), U3.22 (CBUS1)
- new net: D5.2 (A), U3.23 (CBUS0)
- new net: D6.1 (K), R23.1
- new net: D5.1 (K), R22.1
- new net +5V: C17.2, C18.2, R21.1, U3.20 (VCC)
- new net FT_RXD: U3.5 (RXD)
- new net FT_TXD: U3.1 (TXD)
- new net USB_DM: U3.16 (USBD-)
- new net USB_DP: U3.15 (USBD+)

Commit message: V.1.0.4.0_260930
□ PinkBug Lab Study
 - STM32 : 14_E
Parts:
- renumbered C16 to C17, C19 to C18, C17 to C19, C18 to C20, R21 to R29, R22 to R30, R23 to R31, U3 to U4
Connections:
- no-connect marks 0 -> 11
Changed lines of the file:
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@@
 		(color 0 0 0 0)
+	)
+	(no_connect
+		(at 160.02 101.6)
+	)
+	(no_connect
+		(at 160.02 106.68)
+	)
+	(no_connect
+		(at 160.02 86.36)
+	)
+	(no_connect
+		(at 160.02 81.28)
+	)
+	(no_connect
+		(at 160.02 78.74)
+	)
+	(no_connect
+		(at 160.02 104.14)
+	)
+	(no_connect
+		(at 160.02 88.9)
+	)
+	(no_connect
+		(at 119.38 93.98)
+	)
+	(no_connect
+		(at 160.02 76.2)
+	)
+	(no_connect
+		(at 119.38 99.06)
+	)
+	(no_connect
+		(at 160.02 83.82)
 	)
 	(wire
@@
 		(in_pos_files yes)
 		(dnp no)
-		(property "Reference" "#PWR040"
+		(property "Reference" "#PWR049"
 			(at 114.3 118.11 0)
 			(hide yes)
@@
 			(project "stm32f103_t"
 				(path "/85c6611a-7c24-4cf6-98b3-fc639d9f6ec5/89245a68-f20a-4e4a-a4ce-68d3842dae4c"
-					(reference "#PWR040")
+					(reference "#PWR049")
 					(unit 1)
 				)
@@
 		(dnp no)
 		(fields_autoplaced yes)
-		(property "Reference" "C16"
+		(property "Reference" "C17"
 			(at 104.14 49.5299 90)
 			(show_name no)
@@
 			(project "stm32f103_t"
 				(path "/85c6611a-7c24-4cf6-98b3-fc639d9f6ec5/89245a68-f20a-4e4a-a4ce-68d3842dae4c"
-					(reference "C16")
+					(reference "C17")
 					(unit 1)
 				)
@@
 		(in_pos_files yes)
 		(dnp no)
-		(property "Reference" "#PWR045"
+		(property "Reference" "#PWR056"
 			(at 205.74 92.71 0)
 			(hide yes)
@@
 			(project "stm32f103_t"
 				(path "/85c6611a-7c24-4cf6-98b3-fc639d9f6ec5/89245a68-f20a-4e4a-a4ce-68d3842dae4c"
-					(reference "#PWR045")
+					(reference "#PWR056")
 					(unit 1)
 				)
@@
 		(in_pos_files yes)
 		(dnp no)
-		(property "Reference" "#PWR037"
+		(property "Reference" "#PWR048"
 			(at 101.6 64.77 0)
 			(hide yes)
@@
 			(project "stm32f103_t"
 				(path "/85c6611a-7c24-4cf6-98b3-fc639d9f6ec5/89245a68-f20a-4e4a-a4ce-68d3842dae4c"
-					(reference "#PWR037")
+					(reference "#PWR048")
 					(unit 1)
 				)
@@
 		(dnp no)
 		(fields_autoplaced yes)
-		(property "Reference" "U3"
+		(property "Reference" "U4"
 			(at 144.3833 62.23 0)
 			(show_name no)
@@
 			(project "stm32f103_t"
 				(path "/85c6611a-7c24-4cf6-98b3-fc639d9f6ec5/89245a68-f20a-4e4a-a4ce-68d3842dae4c"
-					(reference "U3")
+					(reference "U4")
 					(unit 1)
 				)
@@
 		(in_pos_files yes)
 		(dnp no)
-		(property "Reference" "#PWR042"
+		(property "Reference" "#PWR055"
 			(at 165.1 64.77 0)
 			(hide yes)
@@
 			(project "stm32f103_t"
 				(path "/85c6611a-7c24-4cf6-98b3-fc639d9f6ec5/89245a68-f20a-4e4a-a4ce-68d3842dae4c"
-					(reference "#PWR042")
+					(reference "#PWR055")
 					(unit 1)
 				)
@@
 		(dnp no)
 		(fields_autoplaced yes)
-		(property "Reference" "C18"
+		(property "Reference" "C20"
 			(at 185.42 49.5299 90)
 			(show_name no)
@@
 			(project "stm32f103_t"
 				(path "/85c6611a-7c24-4cf6-98b3-fc639d9f6ec5/89245a68-f20a-4e4a-a4ce-68d3842dae4c"
-					(reference "C18")
+					(reference "C20")
 					(unit 1)
 				)
@@
 		(in_pos_files yes)
 		(dnp no)
-		(property "Reference" "#PWR044"
+		(property "Reference" "#PWR045"
 			(at 90.17 71.12 0)
 			(hide yes)
@@
 			(project "stm32f103_t"
 				(path "/85c6611a-7c24-4cf6-98b3-fc639d9f6ec5/89245a68-f20a-4e4a-a4ce-68d3842dae4c"
-					(reference "#PWR044")
+					(reference "#PWR045")
 					(unit 1)
 				)
@@
 		(in_pos_files yes)
 		(dnp no)
-		(property "Reference" "#PWR039"
+		(property "Reference" "#PWR050"
 			(at 134.62 130.81 0)
 			(hide yes)
@@
 			(project "stm32f103_t"
 				(path "/85c6611a-7c24-4cf6-98b3-fc639d9f6ec5/89245a68-f20a-4e4a-a4ce-68d3842dae4c"
-					(reference "#PWR039")
+					(reference "#PWR050")
 					(unit 1)
 				)
@@
 		(dnp no)
 		(fields_autoplaced yes)
-		(property "Reference" "C17"
+		(property "Reference" "C19"
 			(at 167.64 49.5299 90)
 			(show_name no)
@@
 			(project "stm32f103_t"
 				(path "/85c6611a-7c24-4cf6-98b3-fc639d9f6ec5/89245a68-f20a-4e4a-a4ce-68d3842dae4c"
-					(reference "C17")
+					(reference "C19")
 					(unit 1)
 				)
@@
 		(in_pos_files yes)
 		(dnp no)
-		(property "Reference" "#PWR034"
+		(property "Reference" "#PWR047"
 			(at 101.6 46.99 0)
 			(hide yes)
@@
 			(project "stm32f103_t"
 				(path "/85c6611a-7c24-4cf6-98b3-fc639d9f6ec5/89245a68-f20a-4e4a-a4ce-68d3842dae4c"
-					(reference "#PWR034")
+					(reference "#PWR047")
 					(unit 1)
 				)
@@
 		(in_pos_files yes)
 		(dnp no)
-		(property "Reference" "#PWR036"
+		(property "Reference" "#PWR052"
 			(at 142.24 57.15 0)
 			(hide yes)
@@
 			(project "stm32f103_t"
 				(path "/85c6611a-7c24-4cf6-98b3-fc639d9f6ec5/89245a68-f20a-4e4a-a4ce-68d3842dae4c"
-					(reference "#PWR036")
+					(reference "#PWR052")
 					(unit 1)
 				)
@@
 		(in_pos_files yes)
 		(dnp no)
-		(property "Reference" "R23"
+		(property "Reference" "R31"
 			(at 186.944 97.79 0)
 			(show_name no)
@@
 			(project "stm32f103_t"
 				(path "/85c6611a-7c24-4cf6-98b3-fc639d9f6ec5/89245a68-f20a-4e4a-a4ce-68d3842dae4c"
-					(reference "R23")
+					(reference "R31")
 					(unit 1)
 				)
@@
 		(in_pos_files yes)
 		(dnp no)
-		(property "Reference" "R22"
+		(property "Reference" "R30"
 			(at 186.944 95.25 0)
 			(show_name no)
@@
 			(project "stm32f103_t"
 				(path "/85c6611a-7c24-4cf6-98b3-fc639d9f6ec5/89245a68-f20a-4e4a-a4ce-68d3842dae4c"
-					(reference "R22")
+					(reference "R30")
 					(unit 1)
 				)
@@
 		(in_pos_files yes)
 		(dnp no)
-		(property "Reference" "#PWR038"
+		(property "Reference" "#PWR053"
 			(at 144.78 130.81 0)
 			(hide yes)
@@
 			(project "stm32f103_t"
 				(path "/85c6611a-7c24-4cf6-98b3-fc639d9f6ec5/89245a68-f20a-4e4a-a4ce-68d3842dae4c"
-					(reference "#PWR038")
+					(reference "#PWR053")
 					(unit 1)
 				)
@@
 		(in_pos_files yes)
 		(dnp no)
-		(property "Reference" "#PWR035"
+		(property "Reference" "#PWR051"
 			(at 137.16 57.15 0)
 			(hide yes)
@@
 			(project "stm32f103_t"
 				(path "/85c6611a-7c24-4cf6-98b3-fc639d9f6ec5/89245a68-f20a-4e4a-a4ce-68d3842dae4c"
-					(reference "#PWR035")
+					(reference "#PWR051")
 					(unit 1)
 				)
@@
 		(in_pos_files yes)
 		(dnp no)
-		(property "Reference" "#PWR041"
+		(property "Reference" "#PWR054"
 			(at 165.1 46.99 0)
 			(hide yes)
@@
 			(project "stm32f103_t"
 				(path "/85c6611a-7c24-4cf6-98b3-fc639d9f6ec5/89245a68-f20a-4e4a-a4ce-68d3842dae4c"
-					(reference "#PWR041")
+					(reference "#PWR054")
 					(unit 1)
 				)
@@
 		(in_pos_files yes)
 		(dnp no)
-		(property "Reference" "R21"
+		(property "Reference" "R29"
 			(at 106.68 87.376 0)
 			(show_name no)
@@
 			(project "stm32f103_t"
 				(path "/85c6611a-7c24-4cf6-98b3-fc639d9f6ec5/89245a68-f20a-4e4a-a4ce-68d3842dae4c"
-					(reference "R21")
+					(reference "R29")
 					(unit 1)
 				)
@@
 		(in_pos_files yes)
 		(dnp no)
-		(property "Reference" "C19"
+		(property "Reference" "C18"
 			(at 106.68 68.834 0)
 			(show_name no)
@@
 			(project "stm32f103_t"
 				(path "/85c6611a-7c24-4cf6-98b3-fc639d9f6ec5/89245a68-f20a-4e4a-a4ce-68d3842dae4c"
-					(reference "C19")
+					(reference "C18")
 					(unit 1)
 				)
@@
 		(in_pos_files yes)
 		(dnp no)
-		(property "Reference" "#PWR043"
+		(property "Reference" "#PWR046"
 			(at 100.33 88.9 0)
 			(hide yes)
@@
 			(project "stm32f103_t"
 				(path "/85c6611a-7c24-4cf6-98b3-fc639d9f6ec5/89245a68-f20a-4e4a-a4ce-68d3842dae4c"
-					(reference "#PWR043")
+					(reference "#PWR046")
 					(unit 1)
 				)
