File: circuit/stm32f103_led.kicad_sch (KiCad schematic)
At the start: 8 parts

Commit message: V.1.0.4.0_260930
□ PinkBug Lab Study
 - STM32 : 14_E
Parts:
- renumbered R3 to R13, R4 to R14, R5 to R15, R6 to R16
Changed lines of the file:
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@@
-		)
-	)
-	(label "OUT_LED3"
-		(at 88.9 71.12 180)
-		(effects
-			(font
-				(size 1.27 1.27)
-			)
-			(justify right bottom)
-		)
-	)
-	(label "OUT_LED1"
-		(at 88.9 55.88 180)
-		(effects
-			(font
-				(size 1.27 1.27)
-			)
-			(justify right bottom)
-		)
-	)
-	(label "OUT_LED2"
-		(at 88.9 63.5 180)
-		(effects
-			(font
-				(size 1.27 1.27)
-			)
-			(justify right bottom)
-		)
-	)
-	(label "OUT_LED4"
-		(at 88.9 78.74 180)
-		(effects
-			(font
-				(size 1.27 1.27)
-			)
-			(justify right bottom)
 		)
 	)
@@
 		(in_pos_files yes)
 		(dnp no)
-		(property "Reference" "#PWR016"
+		(property "Reference" "#PWR028"
 			(at 50.8 54.61 0)
 			(hide yes)
@@
 			(project "stm32f103_t"
 				(path "/85c6611a-7c24-4cf6-98b3-fc639d9f6ec5/8f949a12-8888-46cd-a43c-652036d3b159"
-					(reference "#PWR016")
+					(reference "#PWR028")
 					(unit 1)
 				)
@@
 		(in_pos_files yes)
 		(dnp no)
-		(property "Reference" "R3"
+		(property "Reference" "R13"
 			(at 58.42 54.356 0)
 			(show_name no)
@@
 			(project "stm32f103_t"
 				(path "/85c6611a-7c24-4cf6-98b3-fc639d9f6ec5/8f949a12-8888-46cd-a43c-652036d3b159"
-					(reference "R3")
+					(reference "R13")
 					(unit 1)
 				)
@@
 		(in_pos_files yes)
 		(dnp no)
-		(property "Reference" "R5"
+		(property "Reference" "R15"
 			(at 58.42 69.596 0)
 			(show_name no)
@@
 			(project "stm32f103_t"
 				(path "/85c6611a-7c24-4cf6-98b3-fc639d9f6ec5/8f949a12-8888-46cd-a43c-652036d3b159"
-					(reference "R5")
+					(reference "R15")
 					(unit 1)
 				)
@@
 		(in_pos_files yes)
 		(dnp no)
-		(property "Reference" "R6"
+		(property "Reference" "R16"
 			(at 58.42 77.216 0)
 			(show_name no)
@@
 			(project "stm32f103_t"
 				(path "/85c6611a-7c24-4cf6-98b3-fc639d9f6ec5/8f949a12-8888-46cd-a43c-652036d3b159"
-					(reference "R6")
+					(reference "R16")
 					(unit 1)
 				)
@@
 		(in_pos_files yes)
 		(dnp no)
-		(property "Reference" "R4"
+		(property "Reference" "R14"
 			(at 58.42 61.976 0)
 			(show_name no)
@@
 			(project "stm32f103_t"
 				(path "/85c6611a-7c24-4cf6-98b3-fc639d9f6ec5/8f949a12-8888-46cd-a43c-652036d3b159"
-					(reference "R4")
+					(reference "R14")
 					(unit 1)
 				)
