File: circuit/stm32f103_mcu.kicad_sch (KiCad schematic)
At the start: 9 parts, among them SW1 TL1105AF160Q, U1 STM32F103C8T6

Commit message: V.1.0.1.0_260821
□ PinkBug Lab
 - STM32 : 07
Parts:
- added C8, C9: 20pF(2012), 0101_capacitor:c_0805_2012_smd, symbol 0101_capacitor:C
- added J1: PinSocket_1x05, 0501_header_socket:PinSocket_1x05_P2.54mm_Vertical, symbol 0501_header_socket:PinSocket_1x05
- added R1: 0Ω, 0103_resistor:r_0805_2012_smd, symbol 0103_resistor:R
- added R2: 10kΩ, 0103_resistor:r_0805_2012_smd, symbol 0103_resistor:R
- added Y1: SX-1(8.0MHz), 0601_crystal_oscillator:SX-1, symbol 0601_crystal_oscillator:SX-1
- C1, C2, C3, C4, C5, C7: 개정 R.260716.00 -> R.260805.01
- C6: value 1uF(2012) -> 1nF(2012); 개정 R.260716.00 -> R.260805.01
Connections:
- net +3.3V: now also J1.1
- net GND: now also C8.1, C9.2, J1.5, R2.2
- net ~{RST}: now also J1.4
- net SWDIO: now reaches U1.34 (PA13)
- net SWDIO: now also J1.2
- net SWCLK: now reaches U1.37 (PA14)
- net SWCLK: now also J1.3
- net at U1.44 (BOOT0): now also R2.1
- net OSC_IN: now reaches U1.5 (OSC_IN)
- net OSC_IN: now also C9.1, Y1.1
- net at U1.6 (OSC_OUT): now also R1.1
- new net OSC_OUT: C8.2, R1.2, Y1.2
Other:
- note added: "SWD Debug_R.260806.00"

Commit message: V.1.0.2.0_260918
□ PinkBug Lab
 - STM32 : 11
Connections:
- net ADC1_IN1: now reaches U1.10 (PA0-WKUP)
- net ADC1_IN2: now reaches U1.11 (PA1)
- net ADC1_IN3: now reaches U1.12 (PA2)
- net ADC1_IN4: now reaches U1.13 (PA3)
- net IO_IN_SW1: now reaches U1.14 (PA4)
- net IO_IN_SW2: now reaches U1.15 (PA5)
- net IO_IN_SW3: now reaches U1.16 (PA6)
- net IO_IN_SW4: now reaches U1.17 (PA7)
- net MCU_OUT3: now reaches U1.18 (PB0)
- net MCU_OUT4: now reaches U1.19 (PB1)
- net MCU_OUT1: now reaches U1.29 (PA8)
- net MCU_OUT2: now reaches U1.30 (PA9)

Commit message: V.1.0.3.0_260928
□ PinkBug Lab Study
 - STM32 : 13
Parts:
- added R19, R20: 22Ω, 0103_resistor:r_0805_2012_smd, symbol 0103_resistor:R
- added R26, R27: 10kΩ(2012), 0103_resistor:r_0805_2012_smd, symbol 0103_resistor:R
Connections:
- net +3.3V: now also R26.1, R27.1
- net TIM2_CH1_PWM: now reaches U1.38 (PA15)
- net at U1.42 (PB6): now also R19.2
- net at U1.43 (PB7): now also R20.2
- new net MCU_UART1_RX: R20.1, R27.2
- new net MCU_UART1_TX: R19.1, R26.2

Commit message: V.1.0.4.0_260930
□ PinkBug Lab Study
 - STM32 : 14_E
Parts:
- renumbered C4 to C10, C8 to C2, C9 to C3, C1 to C4, C7 to C6, C2 to C7, C6 to C8, C3 to C9, J1 to J3, R20 to R10, R1 to R11, R2 to R12, R26 to R7, R27 to R8, R19 to R9, U1 to U2
Connections:
- net MCU_UART3_TX: now reaches U2.21 (PB10)
- net MCU_UART3_RX: now reaches U2.22 (PB11)
- no-connect marks 0 -> 16
Other:
- moved on the sheet: R7, R8
