File: circuit/stm32f103_pot.kicad_sch (KiCad schematic)
At the start: 12 parts

Commit message: V.1.0.4.0_260930
□ PinkBug Lab Study
 - STM32 : 14_E
Parts:
- renumbered C12 to C13, C13 to C15, C15 to C16, R15 to R25, R17 to R26, R16 to R27, R18 to R28, RV3 to RV2, RV2 to RV3
Changed lines of the file:
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@@
 		(in_pos_files yes)
 		(dnp no)
-		(property "Reference" "#PWR030"
+		(property "Reference" "#PWR040"
 			(at 50.8 120.65 0)
 			(hide yes)
@@
 			(project "stm32f103_t"
 				(path "/85c6611a-7c24-4cf6-98b3-fc639d9f6ec5/8d2be89a-d9ae-4e4d-9900-9269dcf01584"
-					(reference "#PWR030")
+					(reference "#PWR040")
 					(unit 1)
 				)
@@
 		(in_pos_files yes)
 		(dnp no)
-		(property "Reference" "R17"
+		(property "Reference" "R26"
 			(at 60.96 99.822 0)
 			(show_name no)
@@
 			(project "stm32f103_t"
 				(path "/85c6611a-7c24-4cf6-98b3-fc639d9f6ec5/8d2be89a-d9ae-4e4d-9900-9269dcf01584"
-					(reference "R17")
+					(reference "R26")
 					(unit 1)
 				)
@@
 		(in_pos_files yes)
 		(dnp no)
-		(property "Reference" "C13"
+		(property "Reference" "C15"
 			(at 147.066 56.134 90)
 			(show_name no)
@@
 			(project "stm32f103_t"
 				(path "/85c6611a-7c24-4cf6-98b3-fc639d9f6ec5/8d2be89a-d9ae-4e4d-9900-9269dcf01584"
-					(reference "C13")
+					(reference "C15")
 					(unit 1)
 				)
@@
 		(in_pos_files yes)
 		(dnp no)
-		(property "Reference" "#PWR027"
+		(property "Reference" "#PWR041"
 			(at 127 46.99 0)
 			(hide yes)
@@
 			(project "stm32f103_t"
 				(path "/85c6611a-7c24-4cf6-98b3-fc639d9f6ec5/8d2be89a-d9ae-4e4d-9900-9269dcf01584"
-					(reference "#PWR027")
+					(reference "#PWR041")
 					(unit 1)
 				)
@@
 		(in_pos_files yes)
 		(dnp no)
-		(property "Reference" "#PWR028"
+		(property "Reference" "#PWR042"
 			(at 127 69.85 0)
 			(hide yes)
@@
 			(project "stm32f103_t"
 				(path "/85c6611a-7c24-4cf6-98b3-fc639d9f6ec5/8d2be89a-d9ae-4e4d-9900-9269dcf01584"
-					(reference "#PWR028")
+					(reference "#PWR042")
 					(unit 1)
 				)
@@
 		(in_pos_files yes)
 		(dnp no)
-		(property "Reference" "R16"
+		(property "Reference" "R27"
 			(at 137.16 49.022 0)
 			(show_name no)
@@
 			(project "stm32f103_t"
 				(path "/85c6611a-7c24-4cf6-98b3-fc639d9f6ec5/8d2be89a-d9ae-4e4d-9900-9269dcf01584"
-					(reference "R16")
+					(reference "R27")
 					(unit 1)
 				)
@@
 		(in_pos_files yes)
 		(dnp no)
-		(property "Reference" "#PWR026"
+		(property "Reference" "#PWR037"
 			(at 50.8 46.99 0)
 			(hide yes)
@@
 			(project "stm32f103_t"
 				(path "/85c6611a-7c24-4cf6-98b3-fc639d9f6ec5/8d2be89a-d9ae-4e4d-9900-9269dcf01584"
-					(reference "#PWR026")
+					(reference "#PWR037")
 					(unit 1)
 				)
@@
 		(in_pos_files yes)
 		(dnp no)
-		(property "Reference" "R15"
+		(property "Reference" "R25"
 			(at 60.96 49.022 0)
 			(show_name no)
@@
 			(project "stm32f103_t"
 				(path "/85c6611a-7c24-4cf6-98b3-fc639d9f6ec5/8d2be89a-d9ae-4e4d-9900-9269dcf01584"
-					(reference "R15")
+					(reference "R25")
 					(unit 1)
 				)
@@
 		(in_pos_files yes)
 		(dnp no)
-		(property "Reference" "R18"
+		(property "Reference" "R28"
 			(at 137.16 99.822 0)
 			(show_name no)
@@
 			(project "stm32f103_t"
 				(path "/85c6611a-7c24-4cf6-98b3-fc639d9f6ec5/8d2be89a-d9ae-4e4d-9900-9269dcf01584"
-					(reference "R18")
+					(reference "R28")
 					(unit 1)
 				)
@@
 		(dnp no)
 		(fields_autoplaced yes)
-		(property "Reference" "RV3"
+		(property "Reference" "RV2"
 			(at 48.26 100.3299 0)
 			(show_name no)
@@
 			(project "stm32f103_t"
 				(path "/85c6611a-7c24-4cf6-98b3-fc639d9f6ec5/8d2be89a-d9ae-4e4d-9900-9269dcf01584"
-					(reference "RV3")
+					(reference "RV2")
 					(unit 1)
 				)
@@
 		(in_pos_files yes)
 		(dnp no)
-		(property "Reference" "#PWR032"
+		(property "Reference" "#PWR044"
 			(at 127 120.65 0)
 			(hide yes)
@@
 			(project "stm32f103_t"
 				(path "/85c6611a-7c24-4cf6-98b3-fc639d9f6ec5/8d2be89a-d9ae-4e4d-9900-9269dcf01584"
-					(reference "#PWR032")
+					(reference "#PWR044")
 					(unit 1)
 				)
@@
 		(in_pos_files yes)
 		(dnp no)
-		(property "Reference" "#PWR031"
+		(property "Reference" "#PWR043"
 			(at 127 97.79 0)
 			(hide yes)
@@
 			(project "stm32f103_t"
 				(path "/85c6611a-7c24-4cf6-98b3-fc639d9f6ec5/8d2be89a-d9ae-4e4d-9900-9269dcf01584"
-					(reference "#PWR031")
+					(reference "#PWR043")
 					(unit 1)
 				)
@@
 		(in_pos_files yes)
 		(dnp no)
-		(property "Reference" "#PWR029"
+		(property "Reference" "#PWR039"
 			(at 50.8 97.79 0)
 			(hide yes)
@@
 			(project "stm32f103_t"
 				(path "/85c6611a-7c24-4cf6-98b3-fc639d9f6ec5/8d2be89a-d9ae-4e4d-9900-9269dcf01584"
-					(reference "#PWR029")
+					(reference "#PWR039")
 					(unit 1)
 				)
@@
 		(dnp no)
 		(fields_autoplaced yes)
-		(property "Reference" "RV2"
+		(property "Reference" "RV3"
 			(at 124.46 49.5299 0)
 			(show_name no)
@@
 			(project "stm32f103_t"
 				(path "/85c6611a-7c24-4cf6-98b3-fc639d9f6ec5/8d2be89a-d9ae-4e4d-9900-9269dcf01584"
-					(reference "RV2")
+					(reference "RV3")
 					(unit 1)
 				)
@@
 		(in_pos_files yes)
 		(dnp no)
-		(property "Reference" "#PWR025"
+		(property "Reference" "#PWR038"
 			(at 50.8 69.85 0)
 			(hide yes)
@@
 			(project "stm32f103_t"
 				(path "/85c6611a-7c24-4cf6-98b3-fc639d9f6ec5/8d2be89a-d9ae-4e4d-9900-9269dcf01584"
-					(reference "#PWR025")
+					(reference "#PWR038")
 					(unit 1)
 				)
@@
 		(in_pos_files yes)
 		(dnp no)
-		(property "Reference" "C12"
+		(property "Reference" "C13"
 			(at 70.866 56.134 90)
 			(show_name no)
@@
 			(project "stm32f103_t"
 				(path "/85c6611a-7c24-4cf6-98b3-fc639d9f6ec5/8d2be89a-d9ae-4e4d-9900-9269dcf01584"
-					(reference "C12")
+					(reference "C13")
 					(unit 1)
 				)
@@
 		(in_pos_files yes)
 		(dnp no)
-		(property "Reference" "C15"
+		(property "Reference" "C16"
 			(at 147.066 106.934 90)
 			(show_name no)
@@
 			(project "stm32f103_t"
 				(path "/85c6611a-7c24-4cf6-98b3-fc639d9f6ec5/8d2be89a-d9ae-4e4d-9900-9269dcf01584"
-					(reference "C15")
-					(unit 1)
-				)
+					(reference "C16")
+					(unit 1)
+				)
