File: circuit/stm32f103_pwr.kicad_sch (KiCad schematic)
At the start: 3 parts, among them U2 LM1117IMPX-3.3

Commit message: V.1.0.4.0_260930
□ PinkBug Lab Study
 - STM32 : 14_E
Parts:
- renumbered C10 to C11, C11 to C12, U2 to U3
Changed lines of the file:
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@@
 		(in_pos_files yes)
 		(dnp no)
-		(property "Reference" "#PWR012"
+		(property "Reference" "#PWR027"
 			(at 104.14 54.61 0)
 			(hide yes)
@@
 			(project "stm32f103_t"
 				(path "/85c6611a-7c24-4cf6-98b3-fc639d9f6ec5/e25b0e53-e182-4ca1-9f24-21e783ae33ef"
-					(reference "#PWR012")
+					(reference "#PWR027")
 					(unit 1)
 				)
@@
 		(in_pos_files yes)
 		(dnp no)
-		(property "Reference" "C10"
+		(property "Reference" "C11"
 			(at 58.166 56.896 90)
 			(show_name no)
@@
 			(project "stm32f103_t"
 				(path "/85c6611a-7c24-4cf6-98b3-fc639d9f6ec5/e25b0e53-e182-4ca1-9f24-21e783ae33ef"
-					(reference "C10")
+					(reference "C11")
 					(unit 1)
 				)
@@
 		(in_pos_files yes)
 		(dnp no)
-		(property "Reference" "#PWR013"
+		(property "Reference" "#PWR026"
 			(at 96.52 69.85 0)
 			(hide yes)
@@
 			(project "stm32f103_t"
 				(path "/85c6611a-7c24-4cf6-98b3-fc639d9f6ec5/e25b0e53-e182-4ca1-9f24-21e783ae33ef"
-					(reference "#PWR013")
+					(reference "#PWR026")
 					(unit 1)
 				)
@@
 		(dnp no)
 		(fields_autoplaced yes)
-		(property "Reference" "C11"
+		(property "Reference" "C12"
 			(at 99.06 56.934 90)
 			(show_name no)
@@
 			(project "stm32f103_t"
 				(path "/85c6611a-7c24-4cf6-98b3-fc639d9f6ec5/e25b0e53-e182-4ca1-9f24-21e783ae33ef"
-					(reference "C11")
+					(reference "C12")
 					(unit 1)
 				)
@@
 		(in_pos_files yes)
 		(dnp no)
-		(property "Reference" "#PWR015"
+		(property "Reference" "#PWR024"
 			(at 50.8 54.61 0)
 			(hide yes)
@@
 			(project "stm32f103_t"
 				(path "/85c6611a-7c24-4cf6-98b3-fc639d9f6ec5/e25b0e53-e182-4ca1-9f24-21e783ae33ef"
-					(reference "#PWR015")
+					(reference "#PWR024")
 					(unit 1)
 				)
@@
 		(dnp no)
 		(fields_autoplaced yes)
-		(property "Reference" "U2"
+		(property "Reference" "U3"
 			(at 76.2 45.72 0)
 			(show_name no)
@@
 			(project "stm32f103_t"
 				(path "/85c6611a-7c24-4cf6-98b3-fc639d9f6ec5/e25b0e53-e182-4ca1-9f24-21e783ae33ef"
-					(reference "U2")
+					(reference "U3")
 					(unit 1)
 				)
@@
 		(in_pos_files yes)
 		(dnp no)
-		(property "Reference" "#PWR014"
+		(property "Reference" "#PWR025"
 			(at 60.96 69.85 0)
 			(hide yes)
@@
 			(project "stm32f103_t"
 				(path "/85c6611a-7c24-4cf6-98b3-fc639d9f6ec5/e25b0e53-e182-4ca1-9f24-21e783ae33ef"
-					(reference "#PWR014")
-					(unit 1)
-				)
+					(reference "#PWR025")
+					(unit 1)
+				)
