File: circuit/stm32f103_t.kicad_sch (KiCad schematic)
At the start: 0 parts

Commit message: V.1.0.1.0_260821
□ PinkBug Lab
 - STM32 : 07
Other:
- added sheet stm32f103_pwr (stm32f103_pwr.kicad_sch)
Changed lines of the file:
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@@
 	(paper "A4")
 	(sheet
-		(at 38.1 38.1)
+		(at 25.4 25.4)
 		(size 38.1 25.4)
 		(exclude_from_sim no)
@@
 		)
 		(property "Sheetname" "stm32f103_mcu"
-			(at 38.1 37.3884 0)
+			(at 25.4 24.6884 0)
 			(show_name no)
 			(do_not_autoplace no)
@@
 		)
 		(property "Sheetfile" "stm32f103_mcu.kicad_sch"
-			(at 38.1 64.0846 0)
+			(at 25.4 51.3846 0)
 			(show_name no)
 			(do_not_autoplace no)
@@
 				)
 			)
+		)
+	)
+	(sheet
+		(at 76.2 25.4)
+		(size 38.1 25.4)
+		(exclude_from_sim no)
+		(in_bom yes)
+		(on_board yes)
+		(dnp no)
+		(fields_autoplaced yes)
+		(stroke
+			(width 0.1524)
+			(type solid)
+		)
+		(fill
+			(color 0 0 0 0)
+		)
+		(property "Sheetname" "stm32f103_pwr"
+			(at 76.2 24.6884 0)
+			(show_name no)
+			(do_not_autoplace no)
+			(effects
+				(font
+					(size 1.27 1.27)
+				)
+				(justify left bottom)
+			)
+		)
+		(property "Sheetfile" "stm32f103_pwr.kicad_sch"
+			(at 76.2 51.3846 0)
+			(show_name no)
+			(do_not_autoplace no)
+			(effects
+				(font
+					(size 1.27 1.27)
+				)
+				(justify left top)
+			)
+		)
+		(instances
+			(project "stm32f103_t"
+				(path "/85c6611a-7c24-4cf6-98b3-fc639d9f6ec5"
+					(page "3")
+				)
+			)

Commit message: V.1.0.2.0_260918
□ PinkBug Lab
 - STM32 : 11
Other:
- added sheet stm32f103_button (stm32f103_button.kicad_sch)
- added sheet stm32f103_led (stm32f103_led.kicad_sch)
- added sheet stm32f103_pot (stm32f1103_pot.kicad_sch)
- sheet stm32f103_mcu ports: added ADC1_IN1, ADC1_IN2, ADC1_IN3, ADC1_IN4, IO_IN_SW1, IO_IN_SW2, IO_IN_SW3, IO_IN_SW4, MCU_OUT1, MCU_OUT2, MCU_OUT3, MCU_OUT4; removed none

Commit message: V.1.0.3.0_260928
□ PinkBug Lab Study
 - STM32 : 13
Parts:
- added BZ1: GPC1407YB-5V4000, 0605_device:gpc1407yb-5v4000, symbol 0605_device:GPC1407YB-5V4000
- added C20: 0.1uF(2012), 0101_capacitor:c_0805_2012_smd, symbol 0101_capacitor:C
- added J2: 105017-0001, 0503_power:105017-0001, symbol 0503_power:105017-0001
- added Q1: MMBT2222A, 0202_transistor:mmbt2222a, symbol 0202_transistor:MMBT2222A
- added R24: 0Ω(2012), 0103_resistor:r_0805_2012_smd, symbol 0103_resistor:R
- added R25: 1kΩ(2012), 0103_resistor:r_0805_2012_smd, symbol 0103_resistor:R
- added U4: USBLC6-2SC6, 0201_diode:usblc6-2sc6, symbol 0201_diode:USBLC6-2SC6
Connections:
- new net: BZ1.2 (-), Q1.3 (C)
- new net: Q1.1 (B), R25.1
- new net: J2.SH (Shield), R24.2
- new net +3.3V: BZ1.1 (+)
- new net +5V: C20.2, J2.1 (VBUS), U4.5 (VBUS)
- new net BUZZER: R25.2
- new net GND: C20.1, J2.5 (GND), Q1.2 (E), R24.1, U4.2 (GND)
- new net USB_DR_N: U4.3 (I/O2)
- new net USB_DR_P: U4.1 (I/O1)
- new net USB_D_N: J2.2 (D-), U4.4 (I/O2)
- new net USB_D_P: J2.3 (D+), U4.6 (I/O1)
Other:
- added sheet stm32f103_ftdi (stm32f103_ftdi.kicad_sch)
- sheet stm32f103_mcu ports: added MCU_UART1_RX, MCU_UART1_TX, TIM2_CH1_PWM; removed none
- sheet stm32f103_pot: file stm32f1103_pot.kicad_sch -> stm32f103_pot.kicad_sch

Commit message: V.1.0.4.0_260930
□ PinkBug Lab Study
 - STM32 : 14_E
Parts:
- removed J2: 105017-0001, 0503_power:105017-0001, symbol 0503_power:105017-0001
- added H1, H2, H3, H4: MountingHole_Pad, symbol 0602_mechanical_hardware:MountingHole_Pad
- added J1: 105017-0001, 0503_power:105017-0001, symbol 0503_power:105017-0001
- added J2: PinSocket_1x04, 0501_header_socket:pinsocket_1x04_p2.54mm_Vertical, symbol 0501_header_socket:PinSocket_1x04
- added R3, R4, R5, R6: 0Ω(2012), 0103_resistor:r_0805_2012_smd, symbol 0103_resistor:R
- renumbered C20 to C1, R24 to R1, R25 to R2, U4 to U1
Connections:
- net +3.3V: now also J2.1
- net +5V: now also J1.1 (VBUS)
- net GND: now also J1.5 (GND), J2.4, R3.2, R4.2, R5.2, R6.2
- net USB_D_N: now also J1.2 (D-)
- net USB_D_P: now also J1.3 (D+)
- net at R1.2: now also J1.SH (Shield)
- new net: H4.1, R6.1
- new net: H1.1, R3.1
- new net: H2.1, R4.1
- new net: H3.1, R5.1
- new net stm32f103_mcu/MCU_UART3_RX: J2.3
- new net stm32f103_mcu/MCU_UART3_TX: J2.2
- no-connect marks 0 -> 1
Other:
- sheet stm32f103_mcu ports: added MCU_UART3_RX, MCU_UART3_TX; removed none
